File: Schema/Schema.kicad_sch (KiCad schematic)
At the start: 16 parts

Commit message: Added player shooting + collision
Parts:
- added 10uF: C, symbol Device:C
Connections:
- net 5V: now also S1.4; no longer S1.2
- net at A1.18 (D3/PD3), S1.3: now also R1.2, 10uF.1
- net at S1.1: now also 10uF.2; no longer R1.2
Changed lines of the file:
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@@
 	)
 	(junction
+		(at 53.34 48.26)
+		(diameter 0)
+		(color 0 0 0 0)
+	)
+	(junction
 		(at 153.67 72.39)
 		(diameter 0)
@@
 	)
 	(junction
+		(at 53.34 36.83)
+		(diameter 0)
+		(color 0 0 0 0)
+	)
+	(junction
 		(at 135.89 72.39)
 		(diameter 0)
@@
 	(wire
 		(pts
-			(xy 27.94 48.26) (xy 27.94 46.99)
+			(xy 53.34 34.29) (xy 53.34 36.83)
 		)
 		(stroke
@@
 	(wire
 		(pts
+			(xy 44.45 50.8) (xy 50.8 50.8)
+		)
+		(stroke
+			(width 0)
+			(type default)
+		)
+	)
+	(wire
+		(pts
 			(xy 162.56 82.55) (xy 162.56 85.09)
 		)
@@
 	(wire
 		(pts
-			(xy 27.94 36.83) (xy 27.94 39.37)
+			(xy 53.34 24.13) (xy 53.34 26.67)
 		)
 		(stroke
@@
 	(wire
 		(pts
-			(xy 31.75 48.26) (xy 27.94 48.26)
-		)
-		(stroke
-			(width 0)
-			(type default)
-		)
-	)
-	(wire
-		(pts
 			(xy 153.67 59.69) (xy 153.67 62.23)
 		)
@@
 	(wire
 		(pts
-			(xy 25.4 50.8) (xy 31.75 50.8)
+			(xy 44.45 48.26) (xy 53.34 48.26)
 		)
 		(stroke
@@
 	(wire
 		(pts
-			(xy 44.45 48.26) (xy 73.66 48.26)
+			(xy 175.26 50.8) (xy 177.8 50.8)
 		)
 		(stroke
@@
 	(wire
 		(pts
-			(xy 175.26 50.8) (xy 177.8 50.8)
+			(xy 142.24 43.18) (xy 177.8 43.18)
 		)
 		(stroke
@@
 	(wire
 		(pts
-			(xy 142.24 43.18) (xy 177.8 43.18)
+			(xy 53.34 48.26) (xy 73.66 48.26)
 		)
 		(stroke
@@
 	(wire
 		(pts
+			(xy 20.32 48.26) (xy 20.32 36.83)
+		)
+		(stroke
+			(width 0)
+			(type default)
+		)
+	)
+	(wire
+		(pts
+			(xy 20.32 36.83) (xy 53.34 36.83)
+		)
+		(stroke
+			(width 0)
+			(type default)
+		)
+	)
+	(wire
+		(pts
 			(xy 107.95 68.58) (xy 116.84 68.58)
 		)
@@
 	(wire
 		(pts
+			(xy 27.94 48.26) (xy 31.75 48.26)
+		)
+		(stroke
+			(width 0)
+			(type default)
+		)
+	)
+	(wire
+		(pts
 			(xy 162.56 59.69) (xy 162.56 62.23)
 		)
@@
 	(wire
 		(pts
+			(xy 53.34 36.83) (xy 53.34 48.26)
+		)
+		(stroke
+			(width 0)
+			(type default)
+		)
+	)
+	(wire
+		(pts
 			(xy 31.75 115.57) (xy 38.1 115.57)
 		)
@@
 	(global_label "5V"
 		(shape input)
-		(at 25.4 50.8 180)
+		(at 50.8 50.8 0)
 		(fields_autoplaced yes)
 		(effects
@@
 				(size 1.27 1.27)
 			)
-			(justify right)
+			(justify left)
 		)
 		(property "Intersheetrefs" "${INTERSHEET_REFS}"
-			(at 20.1167 50.8 0)
+			(at 56.0833 50.8 0)
 			(effects
 				(font
 					(size 1.27 1.27)
 				)
-				(justify right)
+				(justify left)
 				(hide yes)
 			)
@@
 	)
 	(symbol
+		(lib_id "Device:C")
+		(at 24.13 48.26 90)
+		(unit 1)
+		(exclude_from_sim no)
+		(in_bom yes)
+		(on_board yes)
+		(dnp no)
+		(property "Reference" "10uF"
+			(at 26.416 44.45 90)
+			(effects
+				(font
+					(size 1.27 1.27)
+				)
+				(justify left)
+			)
+		)
+		(property "Value" "C"
+			(at 25.3999 44.45 0)
+			(effects
+				(font
+					(size 1.27 1.27)
+				)
+				(justify left)
+				(hide yes)
+			)
+		)
+		(property "Footprint" ""
+			(at 27.94 47.2948 0)
+			(effects
+				(font
+					(size 1.27 1.27)
+				)
+				(hide yes)
+			)
+		)
+		(property "Datasheet" "~"
+			(at 24.13 48.26 0)
+			(effects
+				(font
+					(size 1.27 1.27)
+				)
+				(hide yes)
+			)
+		)
+		(property "Description" "Unpolarized capacitor"
+			(at 24.13 48.26 0)
+			(effects
+				(font
+					(size 1.27 1.27)
+				)
+				(hide yes)
+			)
+		)
+		(pin "1"
+		)
+		(pin "2"
+		)
+		(instances
+			(project ""
+				(path "/3f91f303-6875-4814-b986-d098b195f512"
+					(reference "10uF")
+					(unit 1)
+				)
+			)
+		)
+	)
+	(symbol
 		(lib_id "PCM_JLCPCB-Resistors:0402,1kΩ")
 		(at 162.56 66.04 0)
@@
 	(symbol
 		(lib_id "PCM_JLCPCB-Resistors:0805,10kΩ")
-		(at 27.94 43.18 0)
+		(at 53.34 30.48 0)
 		(unit 1)
 		(exclude_from_sim no)
@@
 		(fields_autoplaced yes)
 		(property "Reference" "R1"
-			(at 30.48 43.1799 0)
+			(at 55.88 30.4799 0)
 			(effects
 				(font
@@
 		)
 		(property "Value" "10kΩ"
-			(at 27.94 43.18 90)
+			(at 53.34 30.48 90)
 			(do_not_autoplace yes)
 			(effects
@@
 		)
 		(property "Footprint" "PCM_JLCPCB:R_0805"
-			(at 26.162 43.18 90)
+			(at 51.562 30.48 90)
 			(effects
 				(font
@@
 		)
 		(property "Datasheet" "https://www.lcsc.com/datasheet/lcsc_datasheet_2411221126_UNI-ROYAL-Uniroyal-Elec-0805W8F1002T5E_C17414.pdf"
-			(at 27.94 43.18 0)
+			(at 53.34 30.48 0)
 			(effects
 				(font
@@
 		)
 		(property "Description" "125mW Thick Film Resistors 150V ±100ppm/°C ±1% 10kΩ 0805 Chip Resistor - Surface Mount ROHS"
-			(at 27.94 43.18 0)
+			(at 53.34 30.48 0)
 			(effects
 				(font
@@
 		)
 		(property "LCSC" "C17414"
-			(at 27.94 43.18 0)
+			(at 53.34 30.48 0)
 			(effects
 				(font
@@
 		)
 		(property "Stock" "8978117"
-			(at 27.94 43.18 0)
+			(at 53.34 30.48 0)
 			(effects
 				(font
@@
 		)
 		(property "Price" "0.005USD"
-			(at 27.94 43.18 0)
+			(at 53.34 30.48 0)
 			(effects
 				(font
@@
 		)
 		(property "Process" "SMT"
-			(at 27.94 43.18 0)
+			(at 53.34 30.48 0)
 			(effects
 				(font
@@
 		)
 		(property "Minimum Qty" "20"
-			(at 27.94 43.18 0)
+			(at 53.34 30.48 0)
 			(effects
 				(font
@@
 		)
 		(property "Attrition Qty" "10"
-			(at 27.94 43.18 0)
+			(at 53.34 30.48 0)
 			(effects
 				(font
@@
 		)
 		(property "Class" "Basic Component"
-			(at 27.94 43.18 0)
+			(at 53.34 30.48 0)
 			(effects
 				(font
@@
 		)
 		(property "Category" "Resistors,Chip Resistor - Surface Mount"
-			(at 27.94 43.18 0)
+			(at 53.34 30.48 0)
 			(effects
 				(font
@@
 		)
 		(property "Manufacturer" "UNI-ROYAL(Uniroyal Elec)"
-			(at 27.94 43.18 0)
+			(at 53.34 30.48 0)
 			(effects
 				(font
@@
 		)
 		(property "Part" "0805W8F1002T5E"
-			(at 27.94 43.18 0)
+			(at 53.34 30.48 0)
 			(effects
 				(font
@@
 		)
 		(property "Resistance" "10kΩ"
-			(at 27.94 43.18 0)
+			(at 53.34 30.48 0)
 			(effects
 				(font
@@
 		)
 		(property "Power(Watts)" "125mW"
-			(at 27.94 43.18 0)
+			(at 53.34 30.48 0)
 			(effects
 				(font
@@
 		)
 		(property "Type" "Thick Film Resistors"
-			(at 27.94 43.18 0)
+			(at 53.34 30.48 0)
 			(effects
 				(font
@@
 		)
 		(property "Overload Voltage (Max)" "150V"
-			(at 27.94 43.18 0)
+			(at 53.34 30.48 0)
 			(effects
 				(font
@@
 		)
 		(property "Operating Temperature Range" "-55°C~+155°C"
-			(at 27.94 43.18 0)
+			(at 53.34 30.48 0)
 			(effects
 				(font
@@
 		)
 		(property "Tolerance" "±1%"
-			(at 27.94 43.18 0)
+			(at 53.34 30.48 0)
 			(effects
 				(font
@@
 		)
 		(property "Temperature Coefficient" "±100ppm/°C"
-			(at 27.94 43.18 0)
+			(at 53.34 30.48 0)
 			(effects
 				(font
@@
 	(symbol
 		(lib_id "power:GNDREF")
-		(at 27.94 36.83 180)
+		(at 53.34 24.13 180)
 		(unit 1)
 		(exclude_from_sim no)
@@
 		(fields_autoplaced yes)
 		(property "Reference" "#PWR02"
-			(at 27.94 30.48 0)
+			(at 53.34 17.78 0)
 			(effects
 				(font
@@
 		)
 		(property "Value" "GND"
-			(at 27.94 31.75 0)
+			(at 53.34 19.05 0)
 			(effects
 				(font
@@
 		)
 		(property "Footprint" ""
-			(at 27.94 36.83 0)
+			(at 53.34 24.13 0)
 			(effects
 				(font
@@
 		)
 		(property "Datasheet" ""
-			(at 27.94 36.83 0)
+			(at 53.34 24.13 0)
 			(effects
 				(font
@@
 		)
 		(property "Description" "Power symbol creates a global label with name \"GNDREF\" , reference supply ground"
-			(at 27.94 36.83 0)
+			(at 53.34 24.13 0)
 			(effects
 				(font
